File: eagle/ringmod_1496.sch (EAGLE design)
At the start: 28 parts, among them IC1 MC1496, IC2 TL072P, U2 POWER

Commit message: gcode ready
Parts:
- added C4, C6: 100nF, rcl:C-US025-024X044
Connections:
- new net N$21: IC2B.-IN, IC2B.OUT
- net +12V: now also C4.1, IC2P.V+
- net -12V: now also C6.1, IC2P.V-
- net GND: now also C4.2, C6.2, IC2B.+IN
Changed lines of the file:
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@@
 <part name="P+3" library="supply1" deviceset="+12V" device=""/>
 <part name="P+4" library="supply1" deviceset="+12V" device=""/>
+<part name="GND6" library="supply1" deviceset="GND" device=""/>
+<part name="P+5" library="supply1" deviceset="+12V" device=""/>
+<part name="P-4" library="supply1" deviceset="-12V" device=""/>
+<part name="GND7" library="supply1" deviceset="GND" device=""/>
+<part name="C4" library="rcl" deviceset="C-US" device="025-024X044" value="100nF"/>
+<part name="C6" library="rcl" deviceset="C-US" device="025-024X044" value="100nF"/>
 </parts>
 <sheets>
@@
 <instance part="P+3" gate="1" x="116.84" y="71.12"/>
 <instance part="P+4" gate="1" x="121.92" y="66.04"/>
+<instance part="IC2" gate="B" x="144.78" y="81.28"/>
+<instance part="GND6" gate="1" x="129.54" y="81.28"/>
+<instance part="IC2" gate="P" x="137.16" y="2.54"/>
+<instance part="P+5" gate="1" x="137.16" y="15.24"/>
+<instance part="P-4" gate="1" x="137.16" y="-10.16"/>
+<instance part="GND7" gate="1" x="154.94" y="-2.54"/>
+<instance part="C4" gate="G$1" x="144.78" y="10.16" rot="R90"/>
+<instance part="C6" gate="G$1" x="144.78" y="-5.08" rot="R90"/>
 </instances>
 <busses>
@@
 <wire x1="116.84" y1="10.16" x2="116.84" y2="12.7" width="0.1524" layer="91"/>
 </segment>
+<segment>
+<pinref part="IC2" gate="B" pin="+IN"/>
+<pinref part="GND6" gate="1" pin="GND"/>
+<wire x1="137.16" y1="83.82" x2="129.54" y2="83.82" width="0.1524" layer="91"/>
+</segment>
+<segment>
+<pinref part="C4" gate="G$1" pin="2"/>
+<pinref part="GND7" gate="1" pin="GND"/>
+<wire x1="149.86" y1="10.16" x2="154.94" y2="10.16" width="0.1524" layer="91"/>
+<wire x1="154.94" y1="10.16" x2="154.94" y2="2.54" width="0.1524" layer="91"/>
+<wire x1="154.94" y1="2.54" x2="154.94" y2="0" width="0.1524" layer="91"/>
+<wire x1="149.86" y1="-5.08" x2="149.86" y2="2.54" width="0.1524" layer="91"/>
+<wire x1="149.86" y1="2.54" x2="154.94" y2="2.54" width="0.1524" layer="91"/>
+<junction x="154.94" y="2.54"/>
+<pinref part="C6" gate="G$1" pin="2"/>
+</segment>
 </net>
 <net name="+12V" class="0">
@@
 <wire x1="121.92" y1="63.5" x2="121.92" y2="53.34" width="0.1524" layer="91"/>
 </segment>
+<segment>
+<pinref part="IC2" gate="P" pin="V+"/>
+<pinref part="P+5" gate="1" pin="+12V"/>
+<wire x1="137.16" y1="12.7" x2="137.16" y2="10.16" width="0.1524" layer="91"/>
+<pinref part="C4" gate="G$1" pin="1"/>
+<wire x1="142.24" y1="10.16" x2="137.16" y2="10.16" width="0.1524" layer="91"/>
+<junction x="137.16" y="10.16"/>
+</segment>
 </net>
 <net name="-12V" class="0">
@@
 <pinref part="P-3" gate="1" pin="-12V"/>
 <wire x1="88.9" y1="17.78" x2="88.9" y2="20.32" width="0.1524" layer="91"/>
+</segment>
+<segment>
+<pinref part="IC2" gate="P" pin="V-"/>
+<pinref part="P-4" gate="1" pin="-12V"/>
+<wire x1="137.16" y1="-7.62" x2="137.16" y2="-5.08" width="0.1524" layer="91"/>
+<wire x1="142.24" y1="-5.08" x2="137.16" y2="-5.08" width="0.1524" layer="91"/>
+<junction x="137.16" y="-5.08"/>
+<pinref part="C6" gate="G$1" pin="1"/>
 </segment>
 </net>
@@
 </segment>
 </net>
+<net name="N$21" class="0">
+<segment>
+<pinref part="IC2" gate="B" pin="OUT"/>
+<wire x1="152.4" y1="81.28" x2="152.4" y2="73.66" width="0.1524" layer="91"/>
+<pinref part="IC2" gate="B" pin="-IN"/>
+<wire x1="152.4" y1="73.66" x2="137.16" y2="73.66" width="0.1524" layer="91"/>
+<wire x1="137.16" y1="73.66" x2="137.16" y2="78.74" width="0.1524" layer="91"/>
+</segment>
+</net>
